Commit message: Updated the obj file with VHACD collision file

File: src/gym/urdf/arial_vehicle.urdf (robot description, URDF)
Before this commit: robot environment, 1 links, 0 joints
Links:
- link base_link: geometry collision box size=0.1 0.1 0.1; visual box size=0.1 0.1 0.1

File: src/gym/urdf/env.urdf (robot description, URDF)
Before this commit: robot environment, 1 links, 0 joints
Links:
- link base_link: geometry collision mesh filename=meshes/area_collision.obj scale=0.1 0.1 0.1; visual mesh filename=meshes/area_collision.obj scale=0.1 0.1 0.1
