Commit message: Added occupancy plot

File: src/gym/urdf/environment.urdf (robot description, URDF)
Before this commit: robot environment, 6 links, 5 joints
Links:
- removed link block_1
- removed link block_2
- removed link block_3
- removed link block_4
- removed link block_5
- removed link main_building
- added link base_link, mass 1; collision mesh filename=meshes/environment.obj scale=0.1 0.1 0.1; visual mesh filename=meshes/environment.obj scale=0.1 0.1 0.1
Joints:
- removed joint base_link_block_1
- removed joint base_link_block_2
- removed joint base_link_block_3
- removed joint base_link_block_4
- removed joint base_link_block_5

Commit message: Updated roads in environment

File: src/gym/urdf/environment.urdf (robot description, URDF)
Before this commit: robot environment, 1 links, 0 joints
Links:
- removed link base_link
- added link buildings, mass 1; collision mesh filename=meshes/buildings_output_collision.obj scale=0.1 0.1 0.1; visual mesh filename=meshes/buildings.obj scale=0.1 0.1 0.1
- added link roads, mass 1; collision mesh filename=meshes/roads_output_collision.obj scale=0.1 0.1 0.1; visual mesh filename=meshes/roads.obj scale=0.1 0.1 0.1
Joints:
- added joint buildings_roads: type fixed, parent buildings, child roads
