Commit message: Still need to debug

File: src/envs/urdf/arial_vehicle.urdf (robot description, URDF)
Before this commit: robot environment, 1 links, 0 joints
Links:
- link base_link: geometry collision box size=0.5 0.5 0.5; visual box size=0.5 0.5 0.5

File: src/envs/urdf/environment.urdf (robot description, URDF)
Before this commit: robot environment, 2 links, 1 joints
Links:
- removed link roads
- link buildings: geometry collision mesh filename=./meshes/exact_map_output.obj; visual mesh filename=./meshes/exact_map.obj
Joints:
- removed joint buildings_roads

File: src/envs/urdf/ground_vehicle.urdf (robot description, URDF)
Before this commit: robot environment, 1 links, 0 joints
Links:
- link base_link: geometry collision box size=0.5 0.5 0.5; visual box size=0.5 0.5 0.5

Commit message: Formation ,  path planning trivial implementation

File: src/envs/urdf/arial_vehicle.urdf (robot description, URDF)
Before this commit: robot environment, 1 links, 0 joints
Links:
- link base_link: geometry collision sphere radius=0.5; visual sphere radius=0.5
