Commit message: Added textures mesh for the environement

File: src/envs/urdf/environment.urdf (robot description, URDF)
Before this commit: robot environment, 1 links, 0 joints
Links:
- link buildings: geometry collision mesh filename=./meshes/exact_map_output.obj; visual mesh filename=./meshes/benning.obj

File: src/envs/urdf/environment_collision_free.urdf (robot description, URDF)
Before this commit: robot environment, 1 links, 0 joints
Links:
- link buildings: geometry visual mesh filename=./meshes/benning_new.obj
